File: _autosave-ramodeartdmx.kicad_pcb (KiCad board)
At the start: 2 copper layers, 421.9 x 79.2 mm, 28 parts, among them J2 XLR3, J3 XLR3, J4 Conn_01x04_Male, J5 Conn_01x12_Pin, P1 USB_C_Plug_USB2.0, Q1 BC847, Q2 BC847, U1 ESP-12E, U2 AMS1117-3.3, U3 CH340C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

Commit message: (120*80/4)
Parts:
- removed P1: USB_C_Plug_USB2.0, Connector_USB:USB_C_Receptacle_JAE_DX07S016JA1R1500
- added J1: USB_C_Receptacle_USB2.0, usb connectors:TYPE-C-31-M-12, F.Cu at (221.5, 67.6)
- moved Q1 0.13 mm to (199.7, 104.9)
Routing:
- net Net-(U3-UD+): track 45.6 -> 49.5 mm
- net +5V: track 82.3 -> 85.5 mm
- net gnd: track 2.21 -> 4.24 mm
- net tx: track 65.3 -> 66.6 mm
- net gpio0: track 51.0 -> 51.9 mm
Other:
- board size 421.9 x 79.2 mm -> 53.1 x 41.9 mm
